File: hardware/iot_board.kicad_sch (KiCad schematic)
At the start: 19 parts, among them J1 SS-52400-002, J2 B2B-PH-SM4-TB, U1 MCP73871

Commit message: Added a usb_module to the Schematic
Parts:
- added C2, C4: 0.1u, symbol Device:C
- added C3, C5: 10u, symbol Device:C_Polarized
- added LED4: LTST-C170KRKT, LEDC2012X120N, symbol LTST-C170KRKT:LTST-C170KRKT
- added R10: 470, symbol Device:R
- R6: value R -> 20k
Connections:
- net +5V: now also U1.1 (OUT), U1.20 (OUT), VR1.3 (VIN), C4.1, C5.1
- net GND: now also J2.1, VR1.1 (GND), C2.2, C3.2, C4.2, C5.2
- net at LED1.1 (K): now also R7.2; no longer R9.2
- net at LED3.1 (K): now also R9.2; no longer R7.2
- net +3.3V: now reaches VR1.2 (VOUT_2)
- net +3.3V: now also VR1.4 (VOUT_4), C2.1, C3.1, LED4.2 (A)
- new net: LED4.1 (K), R10.2
Other:
- added sheet ESP32-C3-02 (esp32-c3-02.kicad_sch)
- moved on the sheet: J2, LED1, LED2, LED3, VR1

Commit message: Completed the Esp32 schematics
Connections:
- net USB_DN: now also J1.A7 (DN1), J1.B7 (DN2)
- net USB_DP: now also J1.A6 (DP1), J1.B6 (DP2)
- net VBUS: now also J1.A4 (VBUSA1), J1.A9 (VBUSA2), J1.B9 (VBUSB2)
Changed lines of the file:
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@@
 	)
 	(label "VBUS"
-		(at 50.8 58.42 0)
+		(at 57.15 58.42 180)
 		(effects
 			(font
 				(size 1.27 1.27)
 			)
-			(justify left bottom)
+			(justify right bottom)
 		)
 	)
@@
 	)
 	(label "USB_DP"
-		(at 48.26 52.07 0)
+		(at 57.15 50.8 180)
 		(effects
 			(font
 				(size 1.27 1.27)
 			)
-			(justify left bottom)
+			(justify right bottom)
 		)
 	)
 	(label "USB_DN"
-		(at 48.26 54.61 0)
+		(at 57.15 53.34 180)
 		(effects
 			(font
 				(size 1.27 1.27)
 			)
-			(justify left bottom)
+			(justify right bottom)
 		)
 	)
@@
 	)
 	(label "VBUS"
-		(at 99.06 58.42 0)
+		(at 97.79 58.42 0)
 		(effects
 			(font
@@
 	)
 	(label "USB_DP"
-		(at 99.06 52.07 0)
+		(at 97.79 50.8 0)
 		(effects
 			(font
@@
 	)
 	(label "USB_DN"
-		(at 99.06 54.61 0)
+		(at 97.79 53.34 0)
 		(effects
 			(font
@@
 	)
 	(label "VBUS"
-		(at 50.8 45.72 0)
+		(at 57.15 45.72 180)
 		(effects
 			(font
 				(size 1.27 1.27)
 			)
-			(justify left bottom)
+			(justify right bottom)
 		)
 	)

Commit message: Completed Assigning footprints and correcting some mistakes
Parts:
- C1: renamed from C5; footprint (none) -> IOT Board Footprints:T491A
- C2: renamed from C4; footprint (none) -> Capacitor_SMD:C_0805_2012Metric
- C3: renamed from C2; footprint (none) -> Capacitor_SMD:C_0805_2012Metric
- C4: renamed from C1; footprint (none) -> Capacitor_SMD:C_0805_2012Metric
- C5: renamed from C3; footprint (none) -> Resistor_SMD:R_0805_2012Metric
- C6: footprint (none) -> Capacitor_SMD:C_0805_2012Metric
- F1: footprint FUSC3226X100N -> (none)
- LED1: renamed from LED3; footprint LEDC2012X120N -> (none)
- LED2, LED4: footprint LEDC2012X120N -> (none)
- LED3: renamed from LED1; footprint LEDC2012X120N -> (none)
- R1: renamed from R4; footprint (none) -> Resistor_SMD:R_0805_2012Metric
- R10: renamed from R6; footprint (none) -> Resistor_SMD:R_0805_2012Metric
- R2: renamed from R3; footprint (none) -> Resistor_SMD:R_0805_2012Metric
- R3: renamed from R9; footprint (none) -> Resistor_SMD:R_0805_2012Metric
- R4: renamed from R8; footprint (none) -> Resistor_SMD:R_0805_2012Metric
- R5: renamed from R7; footprint (none) -> Resistor_SMD:R_0805_2012Metric
- R6: renamed from R10; footprint (none) -> Resistor_SMD:R_0805_2012Metric
- R7: renamed from R5; footprint (none) -> Resistor_SMD:R_0805_2012Metric
- R8: renamed from R2; footprint (none) -> Resistor_SMD:R_0805_2012Metric
- R9: renamed from R1; footprint (none) -> Resistor_SMD:R_0805_2012Metric
Other:
- note added: "Battery JST Connector"
- note added: "Lipo Battery Charger"
- note added: "Low drop out (LDO) voltage regulator"
- note added: "Power Indicator LED"
- note added: "USB_C connector"
