File: hardware/sensors.kicad_sch (KiCad schematic)
At the start: 0 parts

Commit message: Completed the Sensor Schematics
Parts:
- added C15, C16, C18, C20: 0.1u, symbol Device:C
- added MK1: CMC-5042PF-AC, CMC-5042PF-AC:CUI_CMC-5042PF-AC, symbol CMC-5042PF-AC:CMC-5042PF-AC
- added Q1: TEMT6000X01, TEMT6000X01:TRANS_TEMT6000X01, symbol TEMT6000X01:TEMT6000X01
- added R15, R17: 4K7, symbol Device:R
- added R21, R30: 10K, symbol Device:R
- added R26, R28: 2k, symbol Device:R
- added R27, R29: 1M, symbol Device:R
- added R31: 100K, symbol Device:R
- added U2: BME280, BME280:PSON65P250X250X100-8N, symbol BME280:BME280
- added U7: MAX4466EXK, MAX4466EXK:SOT65P210X110-5N, symbol MAX4466EXK:MAX4466EXK
Connections:
- new net: MK1.OUT, R27.2, R28.2, R29.1, U7.1 (IN+)
- new net: C16.2, R26.2, R28.1
- new net +3.3V: C15.1, C18.1, R15.1, R17.1, R21.1, R26.1, R27.1, U2.2 (CSB), U2.6 (VDDIO), U2.8 (VDD), U7.5 (VCC)
- new net GND: C15.2, C16.1, C18.2, C20.1, MK1.GND, Q1.1, R29.2, R30.1, R30.2, R31.1, U2.1 (GND), U2.5 (SDO), U2.7 (GND), U7.2 (GND), U7.3 (IN-)
- new net MIC_OUT: C20.2, R31.2, U7.4 (OUT)
- new net PHOTO_C: R21.2
- new net SCL: R15.2, U2.4 (SCK)
- new net SDA: R17.2, U2.3 (SDI)

Commit message: Completed Assigning footprints and correcting some mistakes
Parts:
- C15, C16, C18: footprint (none) -> Capacitor_SMD:C_0805_2012Metric
- C17: renamed from C20; footprint (none) -> Capacitor_SMD:C_0805_2012Metric
- R21: renamed from R15; footprint (none) -> Resistor_SMD:R_0805_2012Metric
- R22: renamed from R17; footprint (none) -> Resistor_SMD:R_0805_2012Metric
- R23: renamed from R26; footprint (none) -> Resistor_SMD:R_0805_2012Metric
- R24: renamed from R28; footprint (none) -> Resistor_SMD:R_0805_2012Metric
- R25: renamed from R27; footprint (none) -> Resistor_SMD:R_0805_2012Metric
- R26: renamed from R29; footprint (none) -> Resistor_SMD:R_0805_2012Metric
- R27: renamed from R30; footprint (none) -> Resistor_SMD:R_0805_2012Metric
- R28: renamed from R21; footprint (none) -> Resistor_SMD:R_0805_2012Metric
- R29: renamed from R31; footprint (none) -> Resistor_SMD:R_0805_2012Metric
- renumbered U2 to U6
Other:
- note added: "BME280_sensor"
- note added: "Microphone and amplifier"
- note added: "PHOTO SENSOR"
Changed lines of the file:
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@@
 		)
 	)
+	(text "Microphone and amplifier"
+		(exclude_from_sim no)
+		(at 151.638 88.138 0)
+		(effects
+			(font
+				(size 1.27 1.27)
+			)
+		)
+	)
+	(text "BME280_sensor"
+		(exclude_from_sim no)
+		(at 46.228 36.322 0)
+		(effects
+			(font
+				(size 1.27 1.27)
+			)
+		)
+	)
+	(text "PHOTO SENSOR"
+		(exclude_from_sim no)
+		(at 185.42 38.354 0)
+		(effects
+			(font
+				(size 1.27 1.27)
+			)
+		)
+	)
 	(junction
 		(at 54.61 62.23)
@@
 		)
 	)
-	(label "BME280_sensor"
-		(at 38.1 36.83 0)
-		(effects
-			(font
-				(size 1.27 1.27)
-			)
-			(justify left bottom)
-		)
-	)
-	(label "PHOTO SENSOR"
-		(at 177.8 39.37 0)
-		(effects
-			(font
-				(size 1.27 1.27)
-			)
-			(justify left bottom)
-		)
-	)
-	(label "Microphone and amplifier"
-		(at 139.7 88.9 0)
-		(effects
-			(font
-				(size 1.27 1.27)
-			)
-			(justify left bottom)
-		)
-	)
 	(hierarchical_label "PHOTO_C"
 		(shape input)
@@
 		(dnp no)
 		(fields_autoplaced yes)
-		(property "Reference" "R15"
+		(property "Reference" "R21"
 			(at 57.15 53.3399 0)
 			(show_name no)
@@
 			)
 		)
-		(property "Footprint" ""
+		(property "Footprint" "Resistor_SMD:R_0805_2012Metric"
 			(at 52.832 54.61 90)
 			(hide yes)
@@
 			(project "iot_board"
 				(path "/32f4a40d-6939-405a-8e7e-c6d0e82e69e6/0016dce1-cab5-4d90-b9e5-1e0111bd767f/73ad3676-0386-481c-86e2-4b9b63c0246f"
-					(reference "R15")
+					(reference "R21")
 					(unit 1)
 				)
@@
 		(dnp no)
 		(fields_autoplaced yes)
-		(property "Reference" "R27"
+		(property "Reference" "R25"
 			(at 187.96 118.1099 0)
 			(show_name no)
@@
 			)
 		)
-		(property "Footprint" ""
+		(property "Footprint" "Resistor_SMD:R_0805_2012Metric"
 			(at 183.642 119.38 90)
 			(hide yes)
@@
 			(project "iot_board"
 				(path "/32f4a40d-6939-405a-8e7e-c6d0e82e69e6/0016dce1-cab5-4d90-b9e5-1e0111bd767f/73ad3676-0386-481c-86e2-4b9b63c0246f"
-					(reference "R27")
+					(reference "R25")
 					(unit 1)
 				)
@@
 			)
 		)
-		(property "Footprint" ""
+		(property "Footprint" "Capacitor_SMD:C_0805_2012Metric"
 			(at 253.6952 132.08 0)
 			(hide yes)
@@
 		(dnp no)
 		(fields_autoplaced yes)
-		(property "Reference" "#PWR041"
+		(property "Reference" "#PWR044"
 			(at 215.9 52.07 0)
 			(hide yes)
@@
 			(project "iot_board"
 				(path "/32f4a40d-6939-405a-8e7e-c6d0e82e69e6/0016dce1-cab5-4d90-b9e5-1e0111bd767f/73ad3676-0386-481c-86e2-4b9b63c0246f"
-					(reference "#PWR041")
+					(reference "#PWR044")
 					(unit 1)
 				)
@@
 		(dnp no)
 		(fields_autoplaced yes)
-		(property "Reference" "#PWR045"
+		(property "Reference" "#PWR041"
 			(at 177.8 101.6 0)
 			(hide yes)
@@
 			(project "iot_board"
 				(path "/32f4a40d-6939-405a-8e7e-c6d0e82e69e6/0016dce1-cab5-4d90-b9e5-1e0111bd767f/73ad3676-0386-481c-86e2-4b9b63c0246f"
-					(reference "#PWR045")
+					(reference "#PWR041")
 					(unit 1)
 				)
@@
 		(dnp no)
 		(fields_autoplaced yes)
-		(property "Reference" "R17"
+		(property "Reference" "R22"
 			(at 67.31 53.3399 0)
 			(show_name no)
@@
 			)
 		)
-		(property "Footprint" ""
+		(property "Footprint" "Resistor_SMD:R_0805_2012Metric"
 			(at 62.992 54.61 90)
 			(hide yes)
@@
 			(project "iot_board"
 				(path "/32f4a40d-6939-405a-8e7e-c6d0e82e69e6/0016dce1-cab5-4d90-b9e5-1e0111bd767f/73ad3676-0386-481c-86e2-4b9b63c0246f"
-					(reference "R17")
+					(reference "R22")
 					(unit 1)
 				)
@@
 			)
 		)
-		(property "Footprint" ""
+		(property "Footprint" "Capacitor_SMD:C_0805_2012Metric"
 			(at 119.0752 66.04 0)
 			(hide yes)
@@
 		(in_pos_files yes)
 		(dnp no)
-		(property "Reference" "C20"
+		(property "Reference" "C17"
 			(at 231.902 154.686 90)
 			(show_name no)
@@
 			)
 		)
-		(property "Footprint" ""
+		(property "Footprint" "Capacitor_SMD:C_0805_2012Metric"
 			(at 234.95 150.1648 0)
 			(hide yes)
@@
 			(project "iot_board"
 				(path "/32f4a40d-6939-405a-8e7e-c6d0e82e69e6/0016dce1-cab5-4d90-b9e5-1e0111bd767f/73ad3676-0386-481c-86e2-4b9b63c0246f"
-					(reference "C20")
+					(reference "C17")
 					(unit 1)
 				)
@@
 			)
 		)
-		(property "Footprint" ""
+		(property "Footprint" "Capacitor_SMD:C_0805_2012Metric"
 			(at 166.37 112.0648 0)
 			(hide yes)
@@
 		(dnp no)
 		(fields_autoplaced yes)
-		(property "Reference" "R28"
+		(property "Reference" "R24"
 			(at 173.99 116.8399 0)
 			(show_name no)
@@
 			)
 		)
-		(property "Footprint" ""
+		(property "Footprint" "Resistor_SMD:R_0805_2012Metric"
 			(at 169.672 118.11 90)
 			(hide yes)
@@
 			(project "iot_board"
 				(path "/32f4a40d-6939-405a-8e7e-c6d0e82e69e6/0016dce1-cab5-4d90-b9e5-1e0111bd767f/73ad3676-0386-481c-86e2-4b9b63c0246f"
-					(reference "R28")
+					(reference "R24")
 					(unit 1)
 				)
@@
 		(dnp no)
 		(fields_autoplaced yes)
-		(property "Reference" "U2"
+		(property "Reference" "U6"
 			(at 100.33 44.45 0)
 			(show_name no)
@@
 			(project "iot_board"
 				(path "/32f4a40d-6939-405a-8e7e-c6d0e82e69e6/0016dce1-cab5-4d90-b9e5-1e0111bd767f/73ad3676-0386-481c-86e2-4b9b63c0246f"
-					(reference "U2")
+					(reference "U6")
 					(unit 1)
 				)
@@
 		(dnp no)
 		(fields_autoplaced yes)
-		(property "Reference" "#PWR043"
+		(property "Reference" "#PWR046"
 			(at 252.73 144.78 0)
 			(hide yes)
@@
 			(project "iot_board"
 				(path "/32f4a40d-6939-405a-8e7e-c6d0e82e69e6/0016dce1-cab5-4d90-b9e5-1e0111bd767f/73ad3676-0386-481c-86e2-4b9b63c0246f"
-					(reference "#PWR043")
+					(reference "#PWR046")
 					(unit 1)
 				)
@@
 		(dnp no)
 		(fields_autoplaced yes)
-		(property "Reference" "R21"
+		(property "Reference" "R28"
 			(at 218.44 54.6099 0)
 			(show_name no)
@@
 			)
 		)
-		(property "Footprint" ""
+		(property "Footprint" "Resistor_SMD:R_0805_2012Metric"
 			(at 214.122 55.88 90)
 			(hide yes)
@@
 			(project "iot_board"
 				(path "/32f4a40d-6939-405a-8e7e-c6d0e82e69e6/0016dce1-cab5-4d90-b9e5-1e0111bd767f/73ad3676-0386-481c-86e2-4b9b63c0246f"
-					(reference "R21")
+					(reference "R28")
 					(unit 1)
 				)
@@
 		(dnp no)
 		(fields_autoplaced yes)
-		(property "Reference" "#PWR044"
+		(property "Reference" "#PWR043"
 			(at 204.47 154.94 0)
 			(hide yes)
@@
 			(project "iot_board"
 				(path "/32f4a40d-6939-405a-8e7e-c6d0e82e69e6/0016dce1-cab5-4d90-b9e5-1e0111bd767f/73ad3676-0386-481c-86e2-4b9b63c0246f"
-					(reference "#PWR044")
+					(reference "#PWR043")
 					(unit 1)
 				)
@@
 		(in_pos_files yes)
 		(dnp no)
-		(property "Reference" "R31"
+		(property "Reference" "R29"
 			(at 230.632 140.208 90)
 			(show_name no)
@@
 			)
 		)
-		(property "Footprint" ""
+		(property "Footprint" "Resistor_SMD:R_0805_2012Metric"
 			(at 231.14 146.558 90)
 			(hide yes)
@@
 			(project "iot_board"
 				(path "/32f4a40d-6939-405a-8e7e-c6d0e82e69e6/0016dce1-cab5-4d90-b9e5-1e0111bd767f/73ad3676-0386-481c-86e2-4b9b63c0246f"
-					(reference "R31")
+					(reference "R29")
 					(unit 1)
 				)
@@
 		(dnp no)
 		(fields_autoplaced yes)
-		(property "Reference" "R30"
+		(property "Reference" "R27"
 			(at 203.2 134.6199 0)
 			(show_name no)
@@
 			)
 		)
-		(property "Footprint" ""
+		(property "Footprint" "Resistor_SMD:R_0805_2012Metric"
 			(at 198.882 135.89 90)
 			(hide yes)
@@
 			(project "iot_board"
 				(path "/32f4a40d-6939-405a-8e7e-c6d0e82e69e6/0016dce1-cab5-4d90-b9e5-1e0111bd767f/73ad3676-0386-481c-86e2-4b9b63c0246f"
-					(reference "R30")
+					(reference "R27")
 					(unit 1)
 				)
@@
 		(dnp no)
 		(fields_autoplaced yes)
-		(property "Reference" "#PWR046"
+		(property "Reference" "#PWR040"
 			(at 151.13 119.38 0)
 			(hide yes)
@@
 			(project "iot_board"
 				(path "/32f4a40d-6939-405a-8e7e-c6d0e82e69e6/0016dce1-cab5-4d90-b9e5-1e0111bd767f/73ad3676-0386-481c-86e2-4b9b63c0246f"
-					(reference "#PWR046")
+					(reference "#PWR040")
 					(unit 1)
 				)
@@
 		(dnp no)
 		(fields_autoplaced yes)
-		(property "Reference" "R26"
+		(property "Reference" "R23"
 			(at 173.99 106.6799 0)
 			(show_name no)
@@
 			)
 		)
-		(property "Footprint" ""
+		(property "Footprint" "Resistor_SMD:R_0805_2012Metric"
 			(at 169.672 107.95 90)
 			(hide yes)
@@
 			(project "iot_board"
 				(path "/32f4a40d-6939-405a-8e7e-c6d0e82e69e6/0016dce1-cab5-4d90-b9e5-1e0111bd767f/73ad3676-0386-481c-86e2-4b9b63c0246f"
-					(reference "R26")
+					(reference "R23")
 					(unit 1)
 				)
@@
 		(dnp no)
 		(fields_autoplaced yes)
-		(property "Reference" "#PWR040"
+		(property "Reference" "#PWR042"
 			(at 189.23 74.93 0)
 			(hide yes)
@@
 			(project "iot_board"
 				(path "/32f4a40d-6939-405a-8e7e-c6d0e82e69e6/0016dce1-cab5-4d90-b9e5-1e0111bd767f/73ad3676-0386-481c-86e2-4b9b63c0246f"
-					(reference "#PWR040")
+					(reference "#PWR042")
 					(unit 1)
 				)
@@
 		(dnp no)
 		(fields_autoplaced yes)
-		(property "Reference" "#PWR042"
+		(property "Reference" "#PWR045"
 			(at 252.73 119.38 0)
 			(hide yes)
@@
 			(project "iot_board"
 				(path "/32f4a40d-6939-405a-8e7e-c6d0e82e69e6/0016dce1-cab5-4d90-b9e5-1e0111bd767f/73ad3676-0386-481c-86e2-4b9b63c0246f"
-					(reference "#PWR042")
+					(reference "#PWR045")
 					(unit 1)
 				)
@@
 		(dnp no)
 		(fields_autoplaced yes)
-		(property "Reference" "R29"
+		(property "Reference" "R26"
 			(at 187.96 134.6199 0)
 			(show_name no)
@@
 			)
 		)
-		(property "Footprint" ""
+		(property "Footprint" "Resistor_SMD:R_0805_2012Metric"
 			(at 183.642 135.89 90)
 			(hide yes)
@@
 			(project "iot_board"
 				(path "/32f4a40d-6939-405a-8e7e-c6d0e82e69e6/0016dce1-cab5-4d90-b9e5-1e0111bd767f/73ad3676-0386-481c-86e2-4b9b63c0246f"
-					(reference "R29")
+					(reference "R26")
 					(unit 1)
 				)
